File: PCB/PCK-0.kicad_sch (KiCad schematic)
At the start: 102 parts, among them J1 USB_C_Receptacle_USB2.0_16P, J2 BAT+, J3 BAT-, SW1 EN, SW10 5, SW11 M2, SW12 TAB, SW13 Q, SW14 W, SW15 E, SW16 R, SW17 T, SW18 M3, SW19 CAPSLOCK, SW2 BOOT, SW20 A, SW21 S, SW22 D, SW23 F, SW24 G, SW25 M4, SW26 LSHIFT, SW27 Z, SW28 X, SW29 C, SW3 RotaryEncoder_Switch_MP, SW30 V, SW31 SPACE, SW32 M5, SW33 FN, SW34 CTRL, SW35 SUPER, SW36 ALT, SW37 MOD1, SW38 MOD2, SW4 M1, SW5 ESC, SW6 1, SW7 2, SW8 3, SW9 4, U1 NCP1117-3.3_SOT223, U2 NCP1117-3.3_SOT223, U3 USBLC6-2SC6, U4 ESP32-C6-MINI-1, U5 TVS1400DRV

Commit message: pcb start
Parts:
- SW10: renamed from SW12; value TAB -> 2,2
- SW11: renamed from SW19; value CAPSLOCK -> 2,3
- SW12: renamed from SW26; value LSHIFT -> 2,4
- SW13: renamed from SW33; value FN -> 2,5
- SW14: renamed from SW6; value 1 -> 3,1
- SW15: renamed from SW13; value Q -> 3,2
- SW16: renamed from SW20; value A -> 3,3
- SW17: renamed from SW27; value Z -> 3,4
- SW18: renamed from SW34; value CTRL -> 3,5
- SW19: renamed from SW7; value 2 -> 4,1
- SW20: renamed from SW14; value W -> 4,2
- SW21: value S -> 4,3
- SW22: renamed from SW28; value X -> 4,4
- SW23: renamed from SW35; value SUPER -> 4,5
- SW24: renamed from SW8; value 3 -> 5,1
- SW25: renamed from SW15; value E -> 5,2
- SW26: renamed from SW22; value D -> 5,3
- SW27: renamed from SW29; value C -> 5,4
- SW28: renamed from SW36; value ALT -> 5,5
- SW29: renamed from SW9; value 4 -> 6,1
- SW30: renamed from SW16; value R -> 6,2
- SW31: renamed from SW23; value F -> 6,3
- SW32: renamed from SW30; value V -> 6,4
- SW33: renamed from SW37; value MOD1 -> 6,5
- SW34: renamed from SW10; value 5 -> 7,1
- SW35: renamed from SW17; value T -> 7,2
- SW36: renamed from SW24; value G -> 7,3
- SW37: renamed from SW31; value SPACE -> 7,4
- SW38: value MOD2 -> 7,5
- SW4: value M1 -> 1,1
- SW5: renamed from SW11; value M2 -> 1,2
- SW6: renamed from SW18; value M3 -> 1,3
- SW7: renamed from SW25; value M4 -> 1,4
- SW8: renamed from SW32; value M5 -> 1,5
- SW9: renamed from SW5; value ESC -> 2,1
- renumbered C6 to C4, C4 to C5, C5 to C6, D18 to D10, D25 to D11, D32 to D12, D5 to D13, D12 to D14, D19 to D15, D26 to D16, D33 to D17, D6 to D18, D13 to D19, D27 to D21, D34 to D22, D7 to D23, D14 to D24, D21 to D25, D28 to D26, D35 to D27, D8 to D28, D15 to D29, D22 to D30, D29 to D31, D36 to D32, D9 to D33, D16 to D34, D23 to D35, D30 to D36, D10 to D4, D17 to D5, D24 to D6, D31 to D7, D4 to D8, D11 to D9, H3 to H2, H2 to H3, R6 to R3, R7 to R4, R3 to R5, R4 to R6, R5 to R7, SW3 to SW1, SW1 to SW2, SW2 to SW3, U5 to U2, U2 to U3, U3 to U4, U4 to U5
Other:
- moved on the sheet: D10, D11, D12, D13, D14, D15, D16, D17, D18, D19, D20, D21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

Commit message: pcb key layout done
Parts:
- SW4, SW5, SW6, SW7, SW8: footprint Button_Switch_Keyboard:SW_Cherry_MX_1.00u_PCB -> Button_Switch_Keyboard:SW_Cherry_MX_1.50u_PCB
Connections:
- net IO0: now also SW24.1, SW25.1, SW26.1, SW27.1, SW28.1; no longer SW4.1, SW5.1, SW6.1, SW7.1, SW8.1
- net IO1: now also SW29.1, SW30.1, SW31.1, SW32.1, SW33.1; no longer SW10.1, SW11.1, SW12.1, SW13.1, SW9.1
- net IO2: now also SW4.1, SW5.1, SW6.1, SW7.1, SW8.1; no longer SW14.1, SW15.1, SW16.1, SW17.1, SW18.1
- net IO3: now also SW10.1, SW11.1, SW12.1, SW13.1, SW9.1; no longer SW19.1, SW20.1, SW21.1, SW22.1, SW23.1
- net IO4: now also SW14.1, SW15.1, SW16.1, SW17.1, SW18.1; no longer SW24.1, SW25.1, SW26.1, SW27.1, SW28.1
- net IO5: now also SW19.1, SW20.1, SW21.1, SW22.1, SW23.1; no longer SW29.1, SW30.1, SW31.1, SW32.1, SW33.1
Changed lines of the file:
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@@
 		)
 	)
-	(label "IO1"
+	(label "IO3"
 		(at 215.9 16.51 180)
 		(effects
@@
 		)
 	)
-	(label "IO2"
+	(label "IO4"
 		(at 231.14 16.51 180)
 		(effects
@@
 		)
 	)
-	(label "IO5"
+	(label "IO1"
 		(at 276.86 16.51 180)
 		(effects
@@
 		)
 	)
-	(label "IO0"
+	(label "IO2"
 		(at 200.66 16.51 180)
 		(effects
@@
 		)
 	)
-	(label "IO4"
+	(label "IO0"
 		(at 261.62 16.51 180)
 		(effects
@@
 		)
 	)
-	(label "IO3"
+	(label "IO5"
 		(at 246.38 16.51 180)
 		(effects
@@
 			)
 		)
-		(property "Footprint" "Button_Switch_Keyboard:SW_Cherry_MX_1.00u_PCB"
+		(property "Footprint" "Button_Switch_Keyboard:SW_Cherry_MX_1.50u_PCB"
 			(at 201.93 30.48 0)
 			(hide yes)
@@
 			)
 		)
-		(property "Footprint" "Button_Switch_Keyboard:SW_Cherry_MX_1.00u_PCB"
+		(property "Footprint" "Button_Switch_Keyboard:SW_Cherry_MX_1.50u_PCB"
 			(at 201.93 68.58 0)
 			(hide yes)
@@
 			)
 		)
-		(property "Footprint" "Button_Switch_Keyboard:SW_Cherry_MX_1.00u_PCB"
+		(property "Footprint" "Button_Switch_Keyboard:SW_Cherry_MX_1.50u_PCB"
 			(at 201.93 17.78 0)
 			(hide yes)
@@
 			)
 		)
-		(property "Footprint" "Button_Switch_Keyboard:SW_Cherry_MX_1.00u_PCB"
+		(property "Footprint" "Button_Switch_Keyboard:SW_Cherry_MX_1.50u_PCB"
 			(at 201.93 43.18 0)
 			(hide yes)
@@
 			)
 		)
-		(property "Footprint" "Button_Switch_Keyboard:SW_Cherry_MX_1.00u_PCB"
+		(property "Footprint" "Button_Switch_Keyboard:SW_Cherry_MX_1.50u_PCB"
 			(at 201.93 55.88 0)
 			(hide yes)

Commit message: key layout rework
Parts:
- SW33: footprint Button_Switch_Keyboard:SW_Cherry_MX_1.00u_PCB -> Button_Switch_Keyboard:SW_Cherry_MX_1.75u_PCB
Changed lines of the file:
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@@
 			)
 		)
-		(property "Footprint" "Button_Switch_Keyboard:SW_Cherry_MX_1.00u_PCB"
+		(property "Footprint" "Button_Switch_Keyboard:SW_Cherry_MX_1.75u_PCB"
 			(at 278.13 68.58 0)
 			(hide yes)

Commit message: ground plane and some power routing
Connections:
- net IO12: no longer U5.17 (IO12)
- net IO13: no longer U5.18 (IO13)
- net USB_D+: now also U5.18 (IO13)
- net USB_D-: now also U5.17 (IO12)
Changed lines of the file:
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@@
-	(wire
-		(pts
-			(xy 190.5 45.72) (xy 185.42 45.72)
-		)
-		(stroke
-			(width 0)
-			(type default)
-		)
-	)
 	(wire
 		(pts
@@
 	(wire
 		(pts
+			(xy 185.42 45.72) (xy 190.5 45.72)
+		)
+		(stroke
+			(width 0)
+			(type default)
+		)
+	)
+	(wire
+		(pts
 			(xy 44.45 38.1) (xy 46.99 38.1)
 		)
@@
 	(wire
 		(pts
-			(xy 190.5 43.18) (xy 185.42 43.18)
-		)
-		(stroke
-			(width 0)
-			(type default)
-		)
-	)
-	(wire
-		(pts
 			(xy 273.05 60.96) (xy 273.05 73.66)
 		)
@@
 		(pts
 			(xy 30.48 62.23) (xy 29.21 62.23)
+		)
+		(stroke
+			(width 0)
+			(type default)
+		)
+	)
+	(wire
+		(pts
+			(xy 185.42 43.18) (xy 190.5 43.18)
 		)
 		(stroke
@@
 		)
 	)
+	(label "USB_D-"
+		(at 190.5 43.18 180)
+		(effects
+			(font
+				(size 1.27 1.27)
+			)
+			(justify right bottom)
+		)
+	)
 	(label "IO3"
 		(at 215.9 16.51 180)
@@
 		)
 	)
-	(label "IO12"
-		(at 190.5 43.18 180)
-		(effects
-			(font
-				(size 1.27 1.27)
-			)
-			(justify right bottom)
-		)
-	)
 	(label "IO2"
 		(at 149.86 45.72 0)
@@
 		)
 	)
-	(label "IO13"
-		(at 190.5 45.72 180)
-		(effects
-			(font
-				(size 1.27 1.27)
-			)
-			(justify right bottom)
-		)
-	)
 	(label "IO7"
 		(at 149.86 58.42 0)
@@
 		)
 	)
+	(label "USB_D+"
+		(at 190.5 45.72 180)
+		(effects
+			(font
+				(size 1.27 1.27)
+			)
+			(justify right bottom)
+		)
+	)

Commit message: mcu placement rework, power zones
Parts:
- BT1: footprint Diode_SMD:D_0805_2012Metric -> Battery:BatteryHolder_Keystone_1042_1x18650
Connections:
- net Earth_Protective: no longer J1.SH (SHIELD)
- net GND: now also J1.SH (SHIELD)
Changed lines of the file:
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@@
 	)
 	(symbol
+		(lib_id "power:GND")
+		(at 24.13 63.5 0)
+		(unit 1)
+		(body_style 1)
+		(exclude_from_sim no)
+		(in_bom yes)
+		(on_board yes)
+		(in_pos_files yes)
+		(dnp no)
+		(fields_autoplaced yes)
+		(property "Reference" "#PWR024"
+			(at 24.13 69.85 0)
+			(hide yes)
+			(show_name no)
+			(do_not_autoplace no)
+			(effects
+				(font
+					(size 1.27 1.27)
+				)
+			)
+		)
+		(property "Value" "GND"
+			(at 24.13 68.58 0)
+			(show_name no)
+			(do_not_autoplace no)
+			(effects
+				(font
+					(size 1.27 1.27)
+				)
+			)
+		)
+		(property "Footprint" ""
+			(at 24.13 63.5 0)
+			(hide yes)
+			(show_name no)
+			(do_not_autoplace no)
+			(effects
+				(font
+					(size 1.27 1.27)
+				)
+			)
+		)
+		(property "Datasheet" ""
+			(at 24.13 63.5 0)
+			(hide yes)
+			(show_name no)
+			(do_not_autoplace no)
+			(effects
+				(font
+					(size 1.27 1.27)
+				)
+			)
+		)
+		(property "Description" "Power symbol creates a global label with name \"GND\" , ground"
+			(at 24.13 63.5 0)
+			(hide yes)
+			(show_name no)
+			(do_not_autoplace no)
+			(effects
+				(font
+					(size 1.27 1.27)
+				)
+			)
+		)
+		(pin "1"
+		)
+		(instances
+			(project "PCK-0"
+				(path "/a809c93c-d7d1-4001-af5c-24ca3b5c5d40"
+					(reference "#PWR024")
+					(unit 1)
+				)
+			)
+		)
+	)
+	(symbol
 		(lib_id "Device:D")
 		(at 237.49 64.77 90)
@@
 	)
 	(symbol
-		(lib_id "power:Earth_Protective")
-		(at 24.13 63.5 0)
-		(unit 1)
-		(body_style 1)
-		(exclude_from_sim no)
-		(in_bom yes)
-		(on_board yes)
-		(in_pos_files yes)
-		(dnp no)
-		(property "Reference" "#PWR01"
-			(at 24.13 73.66 0)
-			(hide yes)
-			(show_name no)
-			(do_not_autoplace no)
-			(effects
-				(font
-					(size 1.27 1.27)
-				)
-			)
-		)
-		(property "Value" "Earth_Protective"
-			(at 24.13 71.12 0)
-			(show_name no)
-			(do_not_autoplace no)
-			(effects
-				(font
-					(size 1.27 1.27)
-				)
-			)
-		)
-		(property "Footprint" ""
-			(at 24.13 66.04 0)
-			(hide yes)
-			(show_name no)
-			(do_not_autoplace no)
-			(effects
-				(font
-					(size 1.27 1.27)
-				)
-			)
-		)
-		(property "Datasheet" ""
-			(at 24.13 66.04 0)
-			(hide yes)
-			(show_name no)
-			(do_not_autoplace no)
-			(effects
-				(font
-					(size 1.27 1.27)
-				)
-			)
-		)
-		(property "Description" "Power symbol creates a global label with name \"Earth_Protective\""
-			(at 24.13 63.5 0)
-			(hide yes)
-			(show_name no)
-			(do_not_autoplace no)
-			(effects
-				(font
-					(size 1.27 1.27)
-				)
-			)
-		)
-		(pin "1"
-		)
-		(instances
-			(project "PCK-0"
-				(path "/a809c93c-d7d1-4001-af5c-24ca3b5c5d40"
-					(reference "#PWR01")
-					(unit 1)
-				)
-			)
-		)
-	)
-	(symbol
 		(lib_id "Switch:SW_Push")
 		(at 278.13 22.86 0)
@@
 		(in_pos_files yes)
 		(dnp no)
-		(fields_autoplaced yes)
 		(property "Reference" "J1"
 			(at 29.21 15.24 0)
@@
 			)
 		)
-		(property "Footprint" "Diode_SMD:D_0805_2012Metric"
+		(property "Footprint" "Battery:BatteryHolder_Keystone_1042_1x18650"
 			(at 108.966 86.36 90)
 			(hide yes)
