File: PCB/PCK-0.kicad_pcb (KiCad board)
At the start: 4 copper layers, 321.9 x 127 mm, 91 parts, among them J1 USB_C_Receptacle_USB2.0_16P, J4 Conn_01x15, SW1 EN, SW10 1,2, SW11 2,2, SW12 3,2, SW13 4,2, SW14 5,2, SW15 6,2, SW16 1,3, SW17 2,3, SW18 3,3, SW19 4,3, SW2 BOOT, SW20 5,3, SW21 6,3, SW22 1,4, SW23 2,4, SW24 3,4, SW25 4,4, SW26 5,4, SW27 6,4, SW28 1,4, SW29 2,4, SW3 RotaryEncoder_Switch_MP, SW30 3,4, SW31 4,4, SW32 5,4, SW33 6,4, SW4 1,1, SW5 2,1, SW6 3,1, SW7 4,1, SW8 5,1, SW9 6,1, U1 NCP1117-3.3_SOT223, U2 NCP1117-3.3_SOT223, U3 USBLC6-2SC6, U4 ESP32-C6-MINI-1, U5 TVS1400DRV

Commit message: separated control from input pcb
Parts:
- added J5: Conn_01x15_Socket, Connector_PinSocket_1.00mm:PinSocket_1x15_P1.00mm_Vertical, F.Cu at (120.0, 4.10)
- D10, D11, D12, D13, D14, D15, D16, D17, D18, D19, D20, D21, D22, D23, D24, D25, D26, D27, D28, D29, D3, D30, D31, D32, D4, D5, D6, D7, D8, D9: footprint Diode_THT:D_A-405_P2.54mm_Vertical_AnodeUp -> Diode_SMD:D_0805_2012Metric; moved to F.Cu
- H1, H2, H3, H4: footprint MountingHole:MountingHole_3.2mm_M3_Pad -> MountingHole:MountingHole_3.2mm_M3
- moved H4 266.7 mm to (0.00, 0.00)
- moved H1 203.2 mm to (30.0, 75.0)
- moved C6 193.8 mm to (132.1, 25.5)
- moved D1 193.8 mm to (143.1, 1.54)
- moved U4 193.8 mm to (142.6, 16.5)
- moved C3 193.8 mm to (133.1, 41.7)
- moved C4 193.8 mm to (145.6, 44.4)
- moved C5 193.8 mm to (140.1, 0.80)
- moved C7 193.8 mm to (146.0, 0.80)
- moved D2 193.8 mm to (146.0, 2.98)
- moved R1 193.8 mm to (140.4, 31.6)
- moved R2 193.8 mm to (140.4, 27.0)
- moved R3 193.8 mm to (142.7, 8.42)
- moved R5 193.8 mm to (143.5, 5.72)
- moved R7 193.8 mm to (145.0, 5.73)
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Routing:
- net /IO18: track 8.82 -> 56.6 mm
- net /IO14: track 7.99 -> 49.2 mm, vias 1 -> 3
- net /IO22: track 122.5 -> 163.2 mm
- net /IO20: track 14.4 -> 52.8 mm, vias 1 -> 2
- net /IO15: track 7.91 -> 44.6 mm
- net /IO4: track 248.4 -> 282.3 mm
- net /IO3: track 220.7 -> 253.5 mm
- net /IO2: track 201.3 -> 234.2 mm
- net /IO5: track 232.3 -> 265.2 mm
- net GND: track 12.3 -> 42.8 mm
- net /IO23: track 174.4 -> 192.1 mm, vias 2 -> 1
- net /IO0: track 134.5 -> 142.3 mm
- net /IO1: track 152.4 -> 159.7 mm
- net /IO6: track 186.0 -> 193.0 mm
- net /IO21: track 180.7 -> 187.4 mm
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Other:
- board size 321.9 x 127 mm -> 169.2 x 105 mm
