File: PCB/BTK-0.kicad_pcb (KiCad board)
At the start: 4 copper layers, 203.9 x 105 mm, 94 parts, among them J1 USB_C_Receptacle_USB2.0_16P, J6 Conn_01x16_Pin, J7 Conn_01x16_Socket, SW1 EN, SW10 1,2, SW11 2,2, SW12 3,2, SW13 4,2, SW14 5,2, SW15 6,2, SW16 1,3, SW17 2,3, SW18 3,3, SW19 4,3, SW2 BOOT, SW20 5,3, SW21 6,3, SW22 1,4, SW23 2,4, SW24 3,4, SW25 4,4, SW26 5,4, SW27 6,4, SW28 1,4, SW29 2,4, SW3 RotaryEncoder_Switch_MP, SW30 3,4, SW31 4,4, SW32 5,4, SW33 6,4, SW4 1,1, SW5 2,1, SW6 3,1, SW7 4,1, SW8 5,1, SW9 6,1, U1 NCP1117-3.3_SOT223, U2 NCP1117-3.3_SOT223, U3 USBLC6-2SC6, U4 ESP32-C6-MINI-1, U5 TVS1400DRV

Commit message: restart
Parts:
- removed BT1: Battery, Connector_PinHeader_2.54mm:PinHeader_1x02_P2.54mm_Horizontal
- added C10: 4.7u, Capacitor_SMD:C_0402_1005Metric, F.Cu at (13.3, 45.4)
- added C11: 4.7u, Capacitor_SMD:C_0402_1005Metric, F.Cu at (0.25, 39.3)
- added C8: 4.7u, Capacitor_SMD:C_0402_1005Metric, F.Cu at (35.8, 65.6)
- added C9: 4.7u, Capacitor_SMD:C_0402_1005Metric, F.Cu at (13.3, 44.5)
- added D33: LED, LED_SMD:LED_0805_2012Metric, F.Cu at (37.1, 59.6)
- added D34: LED, LED_SMD:LED_0805_2012Metric, F.Cu at (37.1, 62.7)
- added J2: Battery, Connector_PinHeader_2.54mm:PinHeader_1x02_P2.54mm_Horizontal, F.Cu at (32.7, 53.3)
- added R10: 4.7k, Resistor_SMD:R_0805_2012Metric, F.Cu at (32.6, 59.6)
- added R11: 10k, Resistor_SMD:R_0805_2012Metric, F.Cu at (43.7, 60.3)
- added R12: 1k, Resistor_SMD:R_0805_2012Metric, F.Cu at (32.6, 62.5)
- added R13: 1k, Resistor_SMD:R_0805_2012Metric, F.Cu at (32.6, 65.5)
- added R8: 27k, Resistor_SMD:R_0805_2012Metric, F.Cu at (9.12, 42.1)
- added R9: 1.5k, Resistor_SMD:R_0805_2012Metric, F.Cu at (40.7, 60.3)
- added U6: BQ24075RGT, Package_DFN_QFN:VQFN-16-1EP_3x3mm_P0.5mm_EP1.6x1.6mm, F.Cu at (42.3, 65.2)
- R1, R2, R3, R4, R5, R6, R7: footprint Resistor_SMD:R_0603_1608Metric -> Resistor_SMD:R_0805_2012Metric
- SW10, SW11, SW12, SW13, SW14, SW15, SW16, SW17, SW18, SW19, SW20, SW21, SW22, SW23, SW24, SW25, SW26, SW27, SW28, SW29, SW30, SW31, SW32, SW33, SW4, SW5, SW6, SW7, SW8, SW9: footprint KB_SWITCH:SW_MX_reversible -> kb_switch:SW_MX_reversible
Connections:
- C1 pad 1: VBUS -> VCC
- U1 pad 3: VBUS -> VCC
Routing:
- net VCC: track 0.00 -> 13.4 mm
- removed copper zone on F.Cu, net VBAT

Commit message: we're so back
Parts:
- added D5: TXRX_IND, LED_SMD:LED_0805_2012Metric, F.Cu at (0.82, 48.9)
- added R15: 470, Resistor_SMD:R_0805_2012Metric, F.Cu at (6.10, 49.7)
- added R6: 10k, Resistor_SMD:R_0805_2012Metric, F.Cu at (3.00, 32.2)
- C10, C11, C8, C9: footprint Capacitor_SMD:C_0402_1005Metric -> Capacitor_SMD:C_0805_2012Metric
- D3: renamed from D1; value BOOT_IND -> MODE_IND
- D4: renamed from D2; value BOOT_LIGHT -> BOOT_IND
- J1: footprint Connector_USB:USB_C_Receptacle_GCT_USB4105-xx-A_16P_TopMnt_Horizontal -> USB4510_03_1_A:GCT_USB4510-03-1-A_REVA
- J2: footprint Connector_PinHeader_2.54mm:PinHeader_1x02_P2.54mm_Horizontal -> Connector_PinHeader_2.54mm:PinHeader_1x02_P2.54mm_Vertical
- moved R8 49.0 mm to (0.40, 37.3), turned to -90 degrees
- moved U6 47.0 mm to (4.66, 37.0)
- moved C8 44.3 mm to (6.85, 32.1), turned to 0 degrees
- moved R9 41.3 mm to (10.6, 32.1), turned to 180 degrees
- moved R11 40.2 mm to (1.15, 34.6)
- moved D1 38.1 mm to (0.82, 50.9)
- moved D2 36.9 mm to (0.82, 52.9)
- moved R12 29.0 mm to (6.10, 53.7)
- moved R10 28.7 mm to (6.10, 51.7), turned to 180 degrees
- moved J2 21.4 mm to (11.4, 51.9), turned to 90 degrees
- moved C11 20.1 mm to (12.6, 55.2), turned to 0 degrees
- moved U2 19.7 mm to (13.3, 46.0), turned to 0 degrees
- moved R7 13.4 mm to (4.90, 29.4)
- moved C9 10.7 mm to (7.85, 35.3), turned to 90 degrees
- moved C2 10.5 mm to (15.5, 32.1), turned to 180 degrees
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- renumbered D34 to D1, D7 to D10, D8 to D11, D9 to D12, D10 to D13, D11 to D14, D12 to D15, D13 to D16, D14 to D17, D15 to D18, D16 to D19, D33 to D2, D17 to D20, D18 to D21, D19 to D22, D20 to D23, D21 to D24, D22 to D25, D23 to D26, D24 to D27, D25 to D28, D26 to D29, D27 to D30, D28 to D31, D29 to D32, D30 to D33, D31 to D34, D32 to D35, D3 to D6, D4 to D7, D5 to D8, D6 to D9, J6 to J3, J7 to J4, R12 to R10, R10 to R11, R13 to R12, R6 to R13, R7 to R14, R8 to R7, R11 to R8
Connections:
- C1 pad 1: VCC -> VBUS
- C3 pad 1: VBAT -> VCC
- J2 pad 1: unconnected-(J2-Pin_1-Pad1) -> VBAT
- U1 pad 3: VCC -> VBUS
- U2 pad 3: VBAT -> VCC
- U5 pad 4: VBAT -> VBUS
- U5 pad 5: VBAT -> VBUS
- U5 pad 6: VBAT -> VBUS
- U6 pad 15: GND -> Net-(U6-SYSOFF)
- U6 pad 5: VBUS -> VCC
Routing:
- net /IO3: track 0.00 -> 54.7 mm, vias 0 -> 2
- net +3V3: track 60.3 -> 13.1 mm, vias 19 -> 17
- net VBAT: track 0.00 -> 23.7 mm, vias 0 -> 1
- net VCC: track 13.4 -> 34.6 mm, vias 0 -> 3
- net Net-(D2-K): track 0.00 -> 19.2 mm, vias 0 -> 2
- net Net-(D1-K): track 0.00 -> 16.1 mm, vias 0 -> 2
- net Net-(U6-ILIM): track 0.00 -> 6.44 mm
- net GND: track 65.1 -> 59.3 mm, vias 5 -> 21
- net Net-(U6-TMR): track 0.00 -> 5.24 mm
- net Net-(D5-A): track 0.00 -> 3.74 mm
- net Net-(D2-A): track 0.00 -> 3.74 mm
- net Net-(D1-A): track 0.00 -> 3.74 mm
- net Net-(U6-SYSOFF): track 0.00 -> 3.57 mm
- net Net-(U6-TS): track 0.00 -> 2.88 mm
- net /D-: track 12.7 -> 15.4 mm, vias 0 -> 2
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- added copper zone on F.Cu, net VBAT
- added copper zone on F.Cu, net VBUS
- added copper zone on F.Cu, net VCC

Commit message: i hate data collection
Parts:
- moved C1 11.1 mm to (15.4, 51.6)
- moved C10 11.1 mm to (11.2, 51.5)
- moved C2 11.1 mm to (19.8, 42.4)
- moved C3 11.1 mm to (11.2, 54.5)
- moved C4 11.1 mm to (19.8, 51.6)
- moved C5 11.1 mm to (7.60, 5.90)
- moved C6 11.1 mm to (9.57, 30.3)
- moved C7 11.1 mm to (17.2, 5.80)
- moved C8 11.1 mm to (11.1, 42.4)
- moved C9 11.1 mm to (12.1, 45.5)
- moved D1 11.1 mm to (5.10, 61.2)
- moved D2 11.1 mm to (5.10, 63.2)
- moved D3 11.1 mm to (14.4, 6.54)
- moved D4 11.1 mm to (17.2, 7.98)
- moved D5 11.1 mm to (5.09, 59.2)
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Other:
- board size 203.9 x 105 mm -> 261 x 105 mm

Commit message: final DRC fixes
Parts:
- moved D14 42.4 mm to (-89.4, 34.0)
- moved D20 42.4 mm to (-89.4, 53.1)
- moved D26 42.4 mm to (-89.4, 72.1)
- moved D8 42.4 mm to (-89.4, 15.0)
- moved SW11 42.4 mm to (-116.6, 27.1)
- moved SW17 42.4 mm to (-116.6, 46.1)
- moved SW23 42.4 mm to (-116.6, 65.2)
- moved SW5 42.4 mm to (-116.6, 8.05)
- moved D10 42.4 mm to (-51.3, 15.0)
- moved D11 42.4 mm to (-32.2, 17.0)
- moved D16 42.4 mm to (-51.3, 34.0)
- moved D17 42.4 mm to (-32.2, 36.0)
- moved D22 42.4 mm to (-51.3, 53.1)
- moved D23 42.4 mm to (-32.2, 55.1)
- moved D28 42.4 mm to (-51.3, 72.1)
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Routing:
- net Net-(D35-A): track 3.07 -> 14.1 mm
- net Net-(D3-A): track 4.84 -> 1.89 mm
- net GND: track 59.3 -> 61.8 mm, vias 21 -> 37
- net +3V3: track 13.1 -> 14.8 mm
- net Net-(D2-K): track 19.2 -> 20.7 mm
- net VCC: track 34.6 -> 35.8 mm
- net /D+: track 13.7 -> 14.4 mm
- net /D-: track 15.4 -> 15.5 mm, vias 2 -> 0
- added copper zone on B.Cu, net GND
Other:
- board size 261 x 105 mm -> 167.1 x 105 mm
