File: PCB/BTK-0.kicad_sch (KiCad schematic)
At the start: 108 parts, among them J1 USB_C_Receptacle_USB2.0_16P, J2 Battery, J3 Conn_01x16_Pin, J4 Conn_01x16_Socket, SW1 SW_SPDT, SW10 5,1, SW11 6,1, SW12 1,2, SW13 2,2, SW14 3,2, SW15 4,2, SW16 5,2, SW17 6,2, SW18 1,3, SW19 2,3, SW2 SW_SPDT, SW20 3,3, SW21 4,3, SW22 5,3, SW23 6,3, SW24 1,4, SW25 2,4, SW26 3,4, SW27 4,4, SW28 5,4, SW29 6,4, SW3 EN, SW30 1,4, SW31 2,4, SW32 3,4, SW33 4,4, SW34 5,4, SW35 6,4, SW4 BOOT, SW5 RotaryEncoder_Switch_MP, SW6 1,1, SW7 2,1, SW8 3,1, SW9 4,1, U1 NCP1117-3.3_SOT223, U2 USBLC6-2SC6, U3 ESP32-C6-MINI-1, U4 TVS1400DRV, U5 BQ24075RGT

Commit message: fixing rotary encoder pin
Parts:
- SW3: footprint Button_Switch_THT:SW_PUSH_1P1T_6x3.5mm_H4.3_APEM_MJTP1243 -> Button_Switch_THT:SW_Tactile_Straight_KSA0Axx1LFTR
- SW4: footprint Button_Switch_THT:SW_PUSH_1P1T_6x3.5mm_H4.3_APEM_MJTP1243 -> Button_Switch_THT:SW_PUSH_6mm
Connections:
- net GND: now also J3.4 (Pin_4), J4.4 (Pin_4), SW5.C
- removed net IO21: J3.4 (Pin_4), J4.4 (Pin_4), SW5.C, U3.27 (IO21)
- no-connect marks 6 -> 7
