File: PCB/_restore_backup_2026-08-19T17-21-52-701/PCK-0.kicad_pcb (KiCad board)
At the start: 2 copper layers, 328.9 x 128.2 mm, 102 parts, among them J1 USB_C_Receptacle_USB2.0_16P, J2 BAT+, J3 BAT-, SW1 RotaryEncoder_Switch_MP, SW10 2,2, SW11 2,3, SW12 2,4, SW13 2,5, SW14 3,1, SW15 3,2, SW16 3,3, SW17 3,4, SW18 3,5, SW19 4,1, SW2 EN, SW20 4,2, SW21 4,3, SW22 4,4, SW23 4,5, SW24 5,1, SW25 5,2, SW26 5,3, SW27 5,4, SW28 5,5, SW29 6,1, SW3 BOOT, SW30 6,2, SW31 6,3, SW32 6,4, SW33 6,5, SW34 7,1, SW35 7,2, SW36 7,3, SW37 7,4, SW38 7,5, SW4 1,1, SW5 1,2, SW6 1,3, SW7 1,4, SW8 1,5, SW9 2,1, U1 NCP1117-3.3_SOT223, U2 TVS1400DRV, U3 NCP1117-3.3_SOT223, U4 USBLC6-2SC6, U5 ESP32-C6-MINI-1

Commit message: file organization
Connections:
- BT1 pad 2: Earth_Protective -> GND
- C1 pad 2: Earth_Protective -> GND
- C2 pad 2: Earth_Protective -> GND
- C3 pad 2: Earth_Protective -> GND
- C4 pad 1: Earth_Protective -> GND
- C5 pad 2: Earth_Protective -> GND
- C6 pad 2: Earth_Protective -> GND
- C7 pad 2: Earth_Protective -> GND
- J1 pad A1: Earth_Protective -> GND
- J1 pad A12: Earth_Protective -> GND
- J1 pad B1: Earth_Protective -> GND
- J1 pad B12: Earth_Protective -> GND
- J1 pad SH: Earth_Protective -> GND
- J3 pad 1: Earth_Protective -> GND
- R1 pad 2: Earth_Protective -> GND
- R2 pad 2: Earth_Protective -> GND
- SW1 pad MP: Earth_Protective -> GND
- SW1 pad S2: Earth_Protective -> GND
- SW2 pad 1: Earth_Protective -> GND
- SW3 pad 1: Earth_Protective -> GND
- U1 pad 1: Earth_Protective -> GND
- U2 pad 1: Earth_Protective -> GND
- U2 pad 2: Earth_Protective -> GND
- U2 pad 3: Earth_Protective -> GND
- U2 pad 7: Earth_Protective -> GND
- U3 pad 1: Earth_Protective -> GND
- U4 pad 2: Earth_Protective -> GND
- U5 pad 1: Earth_Protective -> GND
- U5 pad 11: Earth_Protective -> GND
- U5 pad 14: Earth_Protective -> GND
- U5 pad 2: Earth_Protective -> GND
- U5 pad 36: Earth_Protective -> GND
- U5 pad 37: Earth_Protective -> GND
- U5 pad 38: Earth_Protective -> GND
- U5 pad 39: Earth_Protective -> GND
- U5 pad 40: Earth_Protective -> GND
- U5 pad 41: Earth_Protective -> GND
- U5 pad 42: Earth_Protective -> GND
- U5 pad 43: Earth_Protective -> GND
- U5 pad 44: Earth_Protective -> GND
- U5 pad 45: Earth_Protective -> GND
- U5 pad 46: Earth_Protective -> GND
- U5 pad 47: Earth_Protective -> GND
- U5 pad 48: Earth_Protective -> GND
- U5 pad 49: Earth_Protective -> GND
- U5 pad 50: Earth_Protective -> GND
- U5 pad 51: Earth_Protective -> GND
- U5 pad 52: Earth_Protective -> GND
- U5 pad 53: Earth_Protective -> GND
Routing:
- net GND: vias 0 -> 2
- net Earth_Protective: vias 78 -> 76
