File: PCB/_restore_backup_2026-08-19T17-21-52-701/PCK-0.kicad_sch (KiCad schematic)
At the start: 102 parts, among them J1 USB_C_Receptacle_USB2.0_16P, J2 BAT+, J3 BAT-, SW1 RotaryEncoder_Switch_MP, SW10 2,2, SW11 2,3, SW12 2,4, SW13 2,5, SW14 3,1, SW15 3,2, SW16 3,3, SW17 3,4, SW18 3,5, SW19 4,1, SW2 EN, SW20 4,2, SW21 4,3, SW22 4,4, SW23 4,5, SW24 5,1, SW25 5,2, SW26 5,3, SW27 5,4, SW28 5,5, SW29 6,1, SW3 BOOT, SW30 6,2, SW31 6,3, SW32 6,4, SW33 6,5, SW34 7,1, SW35 7,2, SW36 7,3, SW37 7,4, SW38 7,5, SW4 1,1, SW5 1,2, SW6 1,3, SW7 1,4, SW8 1,5, SW9 2,1, U1 NCP1117-3.3_SOT223, U2 TVS1400DRV, U3 NCP1117-3.3_SOT223, U4 USBLC6-2SC6, U5 ESP32-C6-MINI-1

Commit message: file organization
Connections:
- net Earth_Protective: no longer BT1.2 (-), C1.2, C2.2, C3.2, C4.1, C5.2, C6.2, C7.2, J1.A1 (GND), J1.A12 (GND), J1.B1 (GND), J1.B12 (GND), J3.1 (Pin_1), R1.2, R2.2, SW1.MP, SW1.S2, SW2.1, SW3.1, U1.1 (GND), U2.1 (GND), U2.2 (GND), U2.3 (GND), U2.7 (GND), U3.1 (GND), U4.2 (GND), U5.1 (GND), U5.11 (GND), U5.14 (GND), U5.2 (GND), U5.36 (GND), U5.37 (GND), U5.38 (GND), U5.39 (GND), U5.40 (GND), U5.41 (GND), U5.42 (GND), U5.43 (GND), U5.44 (GND), U5.45 (GND), U5.46 (GND), U5.47 (GND), U5.48 (GND), U5.49 (GND), U5.50 (GND), U5.51 (GND), U5.52 (GND), U5.53 (GND)
- new net GND: BT1.2 (-), C1.2, C2.2, C3.2, C4.1, C5.2, C6.2, C7.2, J1.A1 (GND), J1.A12 (GND), J1.B1 (GND), J1.B12 (GND), J3.1 (Pin_1), R1.2, R2.2, SW1.MP, SW1.S2, SW2.1, SW3.1, U1.1 (GND), U2.1 (GND), U2.2 (GND), U2.3 (GND), U2.7 (GND), U3.1 (GND), U4.2 (GND), U5.1 (GND), U5.11 (GND), U5.14 (GND), U5.2 (GND), U5.36 (GND), U5.37 (GND), U5.38 (GND), U5.39 (GND), U5.40 (GND), U5.41 (GND), U5.42 (GND), U5.43 (GND), U5.44 (GND), U5.45 (GND), U5.46 (GND), U5.47 (GND), U5.48 (GND), U5.49 (GND), U5.50 (GND), U5.51 (GND), U5.52 (GND), U5.53 (GND)
Changed lines of the file:
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@@
-	)
-	(junction
-		(at 29.21 62.23)
-		(diameter 0)
-		(color 0 0 0 0)
 	)
 	(junction
@@
 	(junction
 		(at 196.85 35.56)
-		(diameter 0)
-		(color 0 0 0 0)
-	)
-	(junction
-		(at 24.13 62.23)
 		(diameter 0)
 		(color 0 0 0 0)
@@
 		)
 		(stroke
-			(width 0)
-			(type default)
-		)
-	)
-	(wire
-		(pts
-			(xy 24.13 62.23) (xy 29.21 62.23)
-		)
-		(stroke
