File: PCB/_restore_backup_2026-08-23T14-25-17-036/PCK-0.kicad_sch (KiCad schematic)
At the start: 93 parts, among them J1 USB_C_Receptacle_USB2.0_16P, J2 BAT+, J3 BAT-, J4 Conn_01x15, SW1 EN, SW10 1,2, SW11 2,2, SW12 3,2, SW13 4,2, SW14 5,2, SW15 6,2, SW16 1,3, SW17 2,3, SW18 3,3, SW19 4,3, SW2 BOOT, SW20 5,3, SW21 6,3, SW22 1,4, SW23 2,4, SW24 3,4, SW25 4,4, SW26 5,4, SW27 6,4, SW28 1,4, SW29 2,4, SW3 RotaryEncoder_Switch_MP, SW30 3,4, SW31 4,4, SW32 5,4, SW33 6,4, SW4 1,1, SW5 2,1, SW6 3,1, SW7 4,1, SW8 5,1, SW9 6,1, U1 NCP1117-3.3_SOT223, U2 NCP1117-3.3_SOT223, U3 USBLC6-2SC6, U4 ESP32-C6-MINI-1, U5 TVS1400DRV

Commit message: reformat + modular control scheme
Parts:
- removed D27, D28, D29, D31, D32: D, Diode_SMD:D_0805_2012Metric, symbol Device:D
- removed SW28: 1,4, kb_switch:Kailh_socket_MX_reversible, symbol Switch:SW_Push
- removed SW29: 2,4, kb_switch:Kailh_socket_MX_reversible, symbol Switch:SW_Push
- removed SW30: 3,4, kb_switch:Kailh_socket_MX_reversible, symbol Switch:SW_Push
- removed SW32: 5,4, kb_switch:Kailh_socket_MX_reversible, symbol Switch:SW_Push
- removed SW33: 6,4, kb_switch:Kailh_socket_MX_reversible, symbol Switch:SW_Push
- added D16, D23, D9: D, Diode_SMD:D_0805_2012Metric, symbol Device:D
- added SW10: 7,1, Button_Switch_Keyboard:SW_Cherry_MX_1.00u_PCB, symbol Switch:SW_Push
- added SW17: 7,2, Button_Switch_Keyboard:SW_Cherry_MX_1.00u_PCB, symbol Switch:SW_Push
- added SW24: 7,3, Button_Switch_Keyboard:SW_Cherry_MX_1.00u_PCB, symbol Switch:SW_Push
- SW11: renamed from SW10; footprint kb_switch:Kailh_socket_MX_reversible -> Button_Switch_Keyboard:SW_Cherry_MX_1.50u_PCB
- SW12: renamed from SW11; footprint kb_switch:Kailh_socket_MX_reversible -> Button_Switch_Keyboard:SW_Cherry_MX_1.00u_PCB
- SW13: renamed from SW12; footprint kb_switch:Kailh_socket_MX_reversible -> Button_Switch_Keyboard:SW_Cherry_MX_1.00u_PCB
- SW14: renamed from SW13; footprint kb_switch:Kailh_socket_MX_reversible -> Button_Switch_Keyboard:SW_Cherry_MX_1.00u_PCB
- SW15: renamed from SW14; footprint kb_switch:Kailh_socket_MX_reversible -> Button_Switch_Keyboard:SW_Cherry_MX_1.00u_PCB
- SW16: renamed from SW15; footprint kb_switch:Kailh_socket_MX_reversible -> Button_Switch_Keyboard:SW_Cherry_MX_1.00u_PCB
- SW18: renamed from SW16; footprint kb_switch:Kailh_socket_MX_reversible -> Button_Switch_Keyboard:SW_Cherry_MX_1.50u_PCB
- SW19: renamed from SW17; footprint kb_switch:Kailh_socket_MX_reversible -> Button_Switch_Keyboard:SW_Cherry_MX_1.00u_PCB
- SW20: renamed from SW18; footprint kb_switch:Kailh_socket_MX_reversible -> Button_Switch_Keyboard:SW_Cherry_MX_1.00u_PCB
- SW21: renamed from SW19; footprint kb_switch:Kailh_socket_MX_reversible -> Button_Switch_Keyboard:SW_Cherry_MX_1.00u_PCB
- SW22: renamed from SW20; footprint kb_switch:Kailh_socket_MX_reversible -> Button_Switch_Keyboard:SW_Cherry_MX_1.00u_PCB
- SW23: renamed from SW21; footprint kb_switch:Kailh_socket_MX_reversible -> Button_Switch_Keyboard:SW_Cherry_MX_1.00u_PCB
- SW25: renamed from SW22; footprint kb_switch:Kailh_socket_MX_reversible -> Button_Switch_Keyboard:SW_Cherry_MX_1.50u_PCB
- SW26: renamed from SW23; footprint kb_switch:Kailh_socket_MX_reversible -> Button_Switch_Keyboard:SW_Cherry_MX_1.00u_PCB
- SW27: renamed from SW24; footprint kb_switch:Kailh_socket_MX_reversible -> Button_Switch_Keyboard:SW_Cherry_MX_1.00u_PCB
- SW28: renamed from SW25; footprint kb_switch:Kailh_socket_MX_reversible -> Button_Switch_Keyboard:SW_Cherry_MX_1.00u_PCB
- SW29: renamed from SW26; footprint kb_switch:Kailh_socket_MX_reversible -> Button_Switch_Keyboard:SW_Cherry_MX_1.00u_PCB
- SW30: renamed from SW27; footprint kb_switch:Kailh_socket_MX_reversible -> Button_Switch_Keyboard:SW_Cherry_MX_1.00u_PCB
- SW31: value 4,4 -> 7,4; footprint kb_switch:Kailh_socket_MX_reversible -> Button_Switch_Keyboard:SW_Cherry_MX_1.00u_PCB
- SW4: footprint kb_switch:Kailh_socket_MX_reversible -> Button_Switch_Keyboard:SW_Cherry_MX_1.50u_PCB
- SW5, SW6, SW7, SW8, SW9: footprint kb_switch:Kailh_socket_MX_reversible -> Button_Switch_Keyboard:SW_Cherry_MX_1.00u_PCB
- renumbered D9 to D10, D10 to D11, D11 to D12, D12 to D13, D13 to D14, D14 to D15, D15 to D17, D16 to D18, D17 to D19, D18 to D20, D19 to D21, D20 to D22, D21 to D24, D22 to D25, D23 to D26, D24 to D27, D25 to D28, D26 to D29
Connections:
- net IO0: now also SW31.1, SW10.1, SW17.1, SW24.1; no longer D3.1 (K), D4.1 (K), D5.1 (K), D6.1 (K), D7.1 (K), D8.1 (K)
- net IO1: now also D3.1 (K), D4.1 (K), D5.1 (K), D6.1 (K), D7.1 (K), D8.1 (K), D9.1 (K); no longer D10.1 (K), D11.1 (K), D12.1 (K), D13.1 (K), D14.1 (K), D15.1 (K)
- net IO2: no longer SW31.1
- net IO21: now also D10.1 (K), D11.1 (K), D12.1 (K), D13.1 (K), D14.1 (K), D15.1 (K), D16.1 (K); no longer D17.1 (K), D18.1 (K), D19.1 (K), D20.1 (K), D21.1 (K), D22.1 (K)
- net IO6: now also D17.1 (K), D18.1 (K), D19.1 (K), D20.1 (K), D21.1 (K), D22.1 (K), D23.1 (K); no longer D24.1 (K), D25.1 (K), D26.1 (K), D27.1 (K), D28.1 (K), D29.1 (K)
- net IO7: now also D24.1 (K), D25.1 (K), D26.1 (K), D27.1 (K), D28.1 (K), D29.1 (K)
- new net: D23.2 (A), SW24.2
- new net: D9.2 (A), SW10.2
- new net: D16.2 (A), SW17.2
