File: PCB/split/BTK-0_input.kicad_pcb (KiCad board)
At the start: 4 copper layers, 139.5 x 105 mm, 66 parts, among them J7 Conn_01x16_Socket, SW10 1,2, SW11 2,2, SW12 3,2, SW13 4,2, SW14 5,2, SW15 6,2, SW16 1,3, SW17 2,3, SW18 3,3, SW19 4,3, SW20 5,3, SW21 6,3, SW22 1,4, SW23 2,4, SW24 3,4, SW25 4,4, SW26 5,4, SW27 6,4, SW28 1,4, SW29 2,4, SW3 RotaryEncoder_Switch_MP, SW30 3,4, SW31 4,4, SW32 5,4, SW33 6,4, SW4 1,1, SW5 2,1, SW6 3,1, SW7 4,1, SW8 5,1, SW9 6,1

Commit message: nothingburger
Other:
- copper layers 4 -> 2
Changed lines of the file:
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@@
 	(layers
 		(0 "F.Cu" signal)
-		(4 "In1.Cu" signal)
-		(6 "In2.Cu" signal)
 		(2 "B.Cu" signal)
 		(9 "F.Adhes" user "F.Adhesive")
@@
 			)
 			(layer "dielectric 1"
-				(type "prepreg")
-				(thickness 0.1)
-				(material "FR4")
-				(epsilon_r 4.5)
-				(loss_tangent 0.02)
-			)
-			(layer "In1.Cu"
-				(type "copper")
-				(thickness 0.035)
-			)
-			(layer "dielectric 2"
 				(type "core")
-				(thickness 1.24)
-				(material "FR4")
-				(epsilon_r 4.5)
-				(loss_tangent 0.02)
-			)
-			(layer "In2.Cu"
-				(type "copper")
-				(thickness 0.035)
-			)
-			(layer "dielectric 3"
-				(type "prepreg")
-				(thickness 0.1)
+				(thickness 1.51)
 				(material "FR4")
 				(epsilon_r 4.5)
@@
 		(capping no)
 		(filling no)
+		(zone_defaults)
 		(pcbplotparams
 			(layerselection 0x00000000_00000000_55555555_5755f5ff)

Commit message: im boutta die son
Parts:
- moved H2 5.38 mm to (117.1, 5.30)
Routing:
- net /IO4: track 276.9 -> 273.7 mm
- net /IO5: track 261.3 -> 258.6 mm
- net /IO0: track 245.7 -> 243.5 mm
- net /IO1: track 225.3 -> 223.5 mm
- net /IO2: track 177.6 -> 176.2 mm
- net /IO7: track 150.6 -> 149.5 mm
- net /IO14: track 142.2 -> 141.5 mm
Other:
- outline, holes or cut-outs redrawn
- copper layers 2 -> 4
