File: test/BTK-1.kicad_pcb (KiCad board)
At the start: 4 copper layers, 203.9 x 105 mm, 94 parts, among them J1 USB_C_Receptacle_USB2.0_16P, J6 Conn_01x16_Pin, J7 Conn_01x16_Socket, SW1 EN, SW10 1,2, SW11 2,2, SW12 3,2, SW13 4,2, SW14 5,2, SW15 6,2, SW16 1,3, SW17 2,3, SW18 3,3, SW19 4,3, SW2 BOOT, SW20 5,3, SW21 6,3, SW22 1,4, SW23 2,4, SW24 3,4, SW25 4,4, SW26 5,4, SW27 6,4, SW28 1,4, SW29 2,4, SW3 RotaryEncoder_Switch_MP, SW30 3,4, SW31 4,4, SW32 5,4, SW33 6,4, SW4 1,1, SW5 2,1, SW6 3,1, SW7 4,1, SW8 5,1, SW9 6,1, U1 NCP1117-3.3_SOT223, U2 NCP1117-3.3_SOT223, U3 USBLC6-2SC6, U4 ESP32-C6-MINI-1, U5 TVS1400DRV

Commit message: im boutta die son
Parts:
- removed H6: MountingHole_Pad, MountingHole:MountingHole_3.2mm_M3_ISO7380
- added BT1: Battery, Connector_PinHeader_2.54mm:PinHeader_1x02_P2.54mm_Horizontal, F.Cu at (116.1, 44.0)
- added H5: MountingHole_Pad, MountingHole:MountingHole_3.2mm_M3_ISO7380, B.Cu at (117.1, 5.30)
- added J1: USB_C_Receptacle_USB2.0_16P, Connector_USB:USB_C_Receptacle_GCT_USB4105-xx-A_16P_TopMnt_Horizontal, B.Cu at (103.5, 29.6)
- added J6: Conn_01x16_Pin, Connector_PinHeader_1.00mm:PinHeader_1x16_P1.00mm_Vertical, B.Cu at (120.1, 28.8)
- added SW1: EN, Button_Switch_THT:SW_PUSH_1P1T_6x3.5mm_H4.3_APEM_MJTP1243, B.Cu at (119.3, -2.30)
- added SW2: BOOT, Button_Switch_THT:SW_PUSH_1P1T_6x3.5mm_H4.3_APEM_MJTP1243, B.Cu at (109.7, -2.30)
- BT1: moved to B.Cu
- moved D11 167.2 mm to (36.6, 29.1)
- moved D14 167.2 mm to (93.8, 31.1)
- moved D17 167.2 mm to (36.6, 48.1)
- moved D20 167.2 mm to (93.8, 50.1)
- moved D23 167.2 mm to (36.6, 67.2)
- moved D26 167.2 mm to (93.8, 69.2)
- moved D5 167.2 mm to (36.6, 10.0)
- moved D8 167.2 mm to (93.8, 12.0)
- moved SW15 167.2 mm to (85.6, 21.1)
- moved SW21 167.2 mm to (85.6, 40.2)
- moved SW27 167.2 mm to (85.6, 59.2)
- moved SW9 167.2 mm to (85.6, 2.10)
- moved D10 167.2 mm to (17.6, 32.1)
- moved D12 167.2 mm to (55.7, 27.1)
- moved D13 167.2 mm to (74.7, 29.1)
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Routing:
- added copper zone on In1.Cu, net +3V3
- added copper zone on B.Cu, net GND
- added copper zone on In2.Cu, net GND
Other:
- board size 203.9 x 105 mm -> 190.2 x 105 mm
